File: object67/object67.kicad_sch (KiCad schematic)
At the start: 0 parts

Commit message: Created subpages
Other:
- added sheet Mixed Signal Main Board (xsp_main.kicad_sch)
- note added: "OBJECT 67"
Changed lines of the file:
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@@
 	(generator_version "9.0")
 	(paper "A4")
+	(text "OBJECT 67"
+		(exclude_from_sim no)
+		(at 143.002 57.912 0)
+		(effects
+			(font
+				(face "DIN 1451 fette Breitschrift 1936")
+				(size 5.08 5.08)
+			)
+		)
+	)
+	(sheet
+		(at 69.85 99.06)
+		(size 44.45 29.21)
+		(exclude_from_sim no)
+		(in_bom yes)
+		(on_board yes)
+		(dnp no)
+		(fields_autoplaced yes)
+		(stroke
+			(width 0.1524)
+			(type solid)
+		)
+		(fill
+			(color 0 0 0 0.0000)
+		)
+		(property "Sheetname" "Mixed Signal Main Board"
+			(at 69.85 98.3484 0)
+			(effects
+				(font
+					(size 1.27 1.27)
+				)
+				(justify left bottom)
+			)
+		)
+		(property "Sheetfile" "xsp_main.kicad_sch"
+			(at 69.85 128.8546 0)
+			(effects
+				(font
+					(size 1.27 1.27)
+				)
+				(justify left top)
+			)
+		)
+		(instances
+			(project "object67"
+				(path "/a52a93a9-ab60-414c-847b-3047ce4056cf"
+					(page "2")
+				)
+			)
+		)
+	)
 	(sheet_instances
 		(path "/"
