File: object67/audio.kicad_sch (KiCad schematic)
At the start: 29 parts, among them IC1 AK4493SEQ, IC2 TAA5242IRGER, IC3 LMK1C1104PWR, Y1 22.5792M, Y2 24.576M

Commit message: Changes
Parts:
- added C1, C25, C26: 10u, symbol Device:C_Small
- added C20, C21: 10u, symbol Device:C_Polarized_Small
- added C22, C23: 0.1u, symbol Device:C_Small
- renumbered C3 to C1, C1 to C2, C4 to C3, C2 to C4
Connections:
- net MLCK_{1} is gone; now on net MLCK_{DAC}: IC1.46 (MCLK)
- net +3.3V: now also IC2.10 (MD4), IC2.12 (MD5), IC2.6 (IOVDD)
- net +3.3VA: now also IC2.23 (AVDD)
- net GNDA: now also IC2.13 (MD0), IC2.19 (VSSA_1), IC2.20 (VSSA_2), IC2.21 (VSSA_3), IC2.22 (VSSA_4), IC2.25 (EP), IC2.26 (VSS_1), IC2.27 (VSS_2), IC2.28 (VSS_3), IC2.29 (VSS_4), IC2.5 (MD6), IC2.7 (MD1), IC2.8 (MD2), IC2.9 (MD3), C20.2, C21.2, C22.1
- net at IC2.1 (DREG): now also C21.1, C22.2
- net GPO_{ADC}: now reaches IC2.11 (GPO)
- net at IC2.15 (IN1P): now also C23.2
- net at IC2.16 (IN1M): now also C25.1
- net at IC2.17 (IN2P): now also C1.1
- net at IC2.18 (IN2M): now also C26.1
- net BICK_{ADC}: now reaches IC2.2 (BCLK)
- net at IC2.24 (VREF): now also C20.1
- net LRCK_{ADC}: now reaches IC2.3 (FSYNC)
- net SDATA_{ADC}: now reaches IC2.4 (DOUT)
- net BICK renamed BICK_{DAC}
- net LRCK renamed LRCK_{DAC}
- net MLCK_{ADC}: no longer names the net of IC3.7 (Y3)
- net SDATA renamed SDATA_{DAC}
- new net Audio_{IN}LN: C25.2
- new net Audio_{IN}LP: C23.1
- new net Audio_{IN}RN: C26.2
- new net Audio_{IN}RP: C1.2
- no-connect marks 5 -> 7
Other:
- removed sheet Analog Frontend
- note added: "(6)"
- note added: "MD0 shorted to ground for target mode."

Commit message: Analog frontend
Parts:
- renumbered C2 to C1, C9 to C10, C10 to C11, C15 to C13, C13 to C14, C16 to C15, C18 to C16, C14 to C18, C4 to C2, C1 to C3, C3 to C4, C11 to C9, C1 to C?, FB2 to FB1, FB1 to FB2
Connections:
- net Audio_{IN}LN renamed AINLN
- net Audio_{IN}LP renamed AINRP
- net Audio_{IN}RN renamed AINRN
- net Audio_{IN}RP renamed AINLP
- net GPO_{ADC} renamed INT_{ADC}
- net PDN renamed PDN_{DAC}

Commit message: KiCad crashed x2
Parts:
- added R33: 10, symbol Device:R_Small
- added U1: RCJ-2223, object67:DUALRCA, symbol object67:RCJ-2223
- gave numbers to parts that had none: 1
Connections:
- net AINLN is gone; now on net GNDA: C25.2
- net AINRN is gone; now on net GNDA: C26.2
- net AINLP: now also U1.P$1 (GND)
- net AINRP: now also U1.P$3 (TOP)
- net GNDA: now also R33.1
- new net: R33.2, U1.P$2 (BTM)

Commit message: Add LDO
Parts:
- added TP10, TP11, TP12, TP13, TP14, TP15, TP16, TP17, TP5, TP6, TP7, TP8, TP9: TestPoint, symbol Connector:TestPoint
Connections:
- net AOUTLN: now also TP6.1
- net AOUTLP: now also TP5.1
- net AOUTRN: now also TP7.1
- net AOUTRP: now also TP8.1
- net BICK_{ADC}: now also TP15.1
- net BICK_{DAC}: now also TP12.1
- net LRCK_{ADC}: now also TP16.1
- net LRCK_{DAC}: now also TP14.1
- net MLCK_{DAC}: now also TP9.1
- net MLCK_{MCU}: now also TP10.1
- net PDN_{DAC}: now also TP11.1
- net SDATA_{ADC}: now also TP17.1
- net SDATA_{DAC}: now also TP13.1

Commit message: Finished layout
Parts:
- removed Y1: 22.5792M, object67:Oscillator_SMD_NDK_NZ2520SDA-4Pin_2.5x2.0mm, symbol object67:NSC5083D-22.5792M
- removed Y2: 24.576M, object67:Oscillator_SMD_NDK_NZ2520SDA-4Pin_2.5x2.0mm, symbol object67:NSC5083D-24.576M
- added C94, C96: 10u, Capacitor_SMD:CP_Elec_5x5.3, symbol Device:C_Polarized_Small
- added C95, C97: 0.1u, Capacitor_SMD:C_0603_1608Metric, symbol Device:C_Small
- added Y3: ASDLJ-E-49.152MHZ-L-R-T, object67:ASDLJE49152MHZLRT, symbol object67:ASDLJ-E-49.152MHZ-L-R-T
- added Y4: ASDLJ-E-45.1584MHz-L-R-T, object67:ASDLJE451584MHzLRT, symbol object67:ASDLJ-E-45.1584MHz-L-R-T
- C1: footprint (none) -> Capacitor_THT:CP_Radial_D8.0mm_P5.00mm
- C10, C11: footprint (none) -> Capacitor_THT:CP_Radial_D5.0mm_P2.00mm
- C12, C13, C2, C4, C8: footprint (none) -> Capacitor_SMD:C_0603_1608Metric
- C14, C18, C20, C21, C7, C9: footprint (none) -> Capacitor_SMD:CP_Elec_4x5.3
- C15, C17, C23, C25, C26, C5, C58: footprint (none) -> Capacitor_SMD:C_1206_3216Metric
- C16, C19, C22, C6: footprint (none) -> Capacitor_SMD:C_0402_1005Metric
- C3: footprint (none) -> Capacitor_THT:CP_Radial_D8.0mm_P3.50mm
- FB1, FB2, FB3: footprint (none) -> Inductor_SMD:L_0603_1608Metric
Connections:
- net +5VA: now also C94.1, C95.1, C96.1, C97.1
- net CLK_44.1_EN: now also Y4.1 (OE)
- net CLK_48_EN: now also Y3.1 (OE)
- net GNDA: now also C94.2, C95.2, C96.2, C97.2, Y3.2 (GND), Y4.2 (GND)
- net at C14.1, C16.1, FB1.1: now also Y4.4 (VDD)
- net at C18.1, C19.1, FB3.1: now also Y3.4 (VDD)
- net CLK_{22.5792M} renamed CLK_{45.1584M}
- net CLK_{45.1584M}: now also Y3.3 (OUTPUT), Y4.3 (OUTPUT)
Other:
- moved on the sheet: C12, C14, C16, C18, C19, C5, C6, C7, C8, C9, FB1

Commit message: Start layout
Parts:
- R1, R2: footprint (none) -> Resistor_SMD:R_0402_1005Metric
- R33: footprint (none) -> Resistor_SMD:R_1206_3216Metric
- TP10, TP11, TP12, TP13, TP14, TP15, TP16, TP17, TP5, TP6, TP7, TP8, TP9: footprint (none) -> TestPoint:TestPoint_Pad_D2.0mm
Changed lines of the file:
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@@
 			)
 		)
-		(property "Footprint" ""
+		(property "Footprint" "TestPoint:TestPoint_Pad_D2.0mm"
 			(at 151.13 124.46 0)
 			(effects
@@
 			)
 		)
-		(property "Footprint" ""
+		(property "Footprint" "TestPoint:TestPoint_Pad_D2.0mm"
 			(at 266.7 34.29 0)
 			(effects
@@
 			)
 		)
-		(property "Footprint" ""
+		(property "Footprint" "TestPoint:TestPoint_Pad_D2.0mm"
 			(at 241.3 247.65 0)
 			(effects
@@
 			)
 		)
-		(property "Footprint" ""
+		(property "Footprint" "Resistor_SMD:R_0402_1005Metric"
 			(at 43.18 254 0)
 			(effects
@@
 			)
 		)
-		(property "Footprint" ""
+		(property "Footprint" "TestPoint:TestPoint_Pad_D2.0mm"
 			(at 156.21 101.6 0)
 			(effects
@@
 			)
 		)
-		(property "Footprint" ""
+		(property "Footprint" "TestPoint:TestPoint_Pad_D2.0mm"
 			(at 151.13 99.06 0)
 			(effects
@@
 			)
 		)
-		(property "Footprint" ""
+		(property "Footprint" "TestPoint:TestPoint_Pad_D2.0mm"
 			(at 158.75 127 0)
 			(effects
@@
 			)
 		)
-		(property "Footprint" ""
+		(property "Footprint" "TestPoint:TestPoint_Pad_D2.0mm"
 			(at 205.74 252.73 0)
 			(effects
@@
 			)
 		)
-		(property "Footprint" ""
+		(property "Footprint" "Resistor_SMD:R_0402_1005Metric"
 			(at 43.18 231.14 0)
 			(effects
@@
 			)
 		)
-		(property "Footprint" ""
+		(property "Footprint" "TestPoint:TestPoint_Pad_D2.0mm"
 			(at 264.16 31.75 0)
 			(effects
@@
 			)
 		)
-		(property "Footprint" ""
+		(property "Footprint" "TestPoint:TestPoint_Pad_D2.0mm"
 			(at 68.5535 101.6 0)
 			(effects
@@
 			)
 		)
-		(property "Footprint" ""
+		(property "Footprint" "Resistor_SMD:R_1206_3216Metric"
 			(at 256.54 118.11 0)
 			(effects
@@
 			)
 		)
-		(property "Footprint" ""
+		(property "Footprint" "TestPoint:TestPoint_Pad_D2.0mm"
 			(at 76.2 106.68 0)
 			(effects
@@
 			)
 		)
-		(property "Footprint" ""
+		(property "Footprint" "TestPoint:TestPoint_Pad_D2.0mm"
 			(at 72.39 104.14 0)
 			(effects
@@
 			)
 		)
-		(property "Footprint" ""
+		(property "Footprint" "TestPoint:TestPoint_Pad_D2.0mm"
 			(at 80.01 109.22 0)
 			(effects
@@
 			)
 		)
-		(property "Footprint" ""
+		(property "Footprint" "TestPoint:TestPoint_Pad_D2.0mm"
 			(at 269.24 36.83 0)
 			(effects

Commit message: Updated pcb
Parts:
- added R46: 22, Capacitor_SMD:C_0201_0603Metric, symbol Device:R_Small
Connections:
- net MLCK_{DAC}: now also R46.1; no longer IC1.46 (MCLK)
- new net: IC1.46 (MCLK), R46.2
- no-connect marks 7 -> 9
Changed lines of the file:
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@@
 	)
 	(no_connect
+		(at 91.44 124.46)
+	)
+	(no_connect
 		(at 91.44 114.3)
 	)
@@
 		(at 232.41 255.27)
 	)
+	(no_connect
+		(at 91.44 121.92)
+	)
 	(wire
 		(pts
@@
 	(wire
 		(pts
+			(xy 104.14 71.12) (xy 104.14 73.66)
+		)
+		(stroke
+			(width 0)
+			(type default)
+		)
+	)
+	(wire
+		(pts
 			(xy 337.82 48.26) (xy 337.82 71.12)
 		)
@@
 	(global_label "MLCK_{DAC}"
 		(shape input)
-		(at 104.14 78.74 90)
+		(at 104.14 71.12 90)
 		(fields_autoplaced yes)
 		(effects
@@
 		)
 		(property "Intersheetrefs" "${INTERSHEET_REFS}"
-			(at 104.14 67.7816 90)
+			(at 104.14 60.1616 90)
 			(effects
 				(font
@@
 					(unit 1)
 				)
+			)
+		)
+	)
+	(symbol
+		(lib_id "Device:R_Small")
+		(at 104.14 76.2 0)
+		(unit 1)
+		(exclude_from_sim no)
+		(in_bom yes)
+		(on_board yes)
+		(dnp no)
+		(property "Reference" "R46"
+			(at 102.362 79.248 0)
+			(effects
+				(font
+					(size 1.016 1.016)
+				)
+				(justify left)
+			)
+		)
+		(property "Value" "22"
+			(at 104.14 77.724 90)
+			(effects
+				(font
+					(size 1.27 1.27)
+				)
+				(justify left)
+			)
+		)
+		(property "Footprint" "Capacitor_SMD:C_0201_0603Metric"
+			(at 104.14 76.2 0)
+			(effects
+				(font
+					(size 1.27 1.27)
+				)
+				(hide yes)
+			)
+		)
+		(property "Datasheet" "~"
+			(at 104.14 76.2 0)
+			(effects
+				(font
+					(size 1.27 1.27)
+				)
+				(hide yes)
+			)
+		)
+		(property "Description" "Resistor, small symbol"
+			(at 104.14 76.2 0)
+			(effects
+				(font
+					(size 1.27 1.27)
+				)
+				(hide yes)
+			)
+		)
+		(pin "1"
+		)
+		(pin "2"
+		)
+		(instances
+			(project ""
+				(path "/a52a93a9-ab60-414c-847b-3047ce4056cf/2d7be8e2-05a1-49f5-8994-604be09973f2/f43f4198-176f-4b92-97fe-5a3f8cda9d3b"
+					(reference "R46")
+					(unit 1)
+				)

Commit message: More layouts
Connections:
- net MLCK_{DAC}: now also IC3.3 (Y0), TP10.1; no longer IC3.8 (Y1), TP9.1
- net MLCK_{MCU}: now also IC3.8 (Y1), TP9.1; no longer IC3.3 (Y0), TP10.1
