File: object67/mcu.kicad_sch (KiCad schematic)
At the start: 0 parts

Commit message: LAyout
Parts:
- added C100, C101, C102, C103, C104, C105, C107, C108, C109, C111, C112, C113, C122, C52, C54: 0.1u, Capacitor_SMD:C_0402_1005Metric, symbol Device:C_Small
- added C114: 10u, Capacitor_SMD:CP_Elec_4x5.3, symbol Device:C_Polarized_Small
- added C115, C116, C123: 2.2u, Capacitor_SMD:C_0603_1608Metric, symbol Device:C_Small
- added C117, C120: 10u, Capacitor_SMD:C_0603_1608Metric, symbol Device:C_Small
- added C118, C119: 0.1u, Capacitor_SMD:C_0603_1608Metric, symbol Device:C_Small
- added C121: 1u, Capacitor_SMD:C_1206_3216Metric, symbol Device:C_Small
- added FB3: 120R, Inductor_SMD:L_0603_1608Metric, symbol Device:FerriteBead_Small
- added J5: Conn_01x16_Socket, Connector_JST:JST_PH_S16B-PH-K_1x16_P2.00mm_Horizontal, symbol Connector:Conn_01x16_Socket
- added J6: Conn_01x08_Pin, Connector_PinHeader_2.54mm:PinHeader_1x08_P2.54mm_Vertical, symbol Connector:Conn_01x08_Pin
- added J7: USB_C_Receptacle_USB2.0_16P, Connector_USB:USB_C_Receptacle_GCT_USB4085, symbol Connector:USB_C_Receptacle_USB2.0_16P
- added J8: Conn_01x04_Pin, Connector_PinHeader_2.54mm:PinHeader_1x04_P2.54mm_Vertical, symbol Connector:Conn_01x04_Pin
- added JP1: Boot0, Jumper:SolderJumper-2_P1.3mm_Open_RoundedPad1.0x1.5mm, symbol Jumper:SolderJumper_2_Open
- added JP2: NRST, Jumper:SolderJumper-2_P1.3mm_Open_RoundedPad1.0x1.5mm, symbol Jumper:SolderJumper_2_Open
- added R47: 10k, Resistor_SMD:R_0603_1608Metric, symbol Device:R_Small
- added R49, R50, R51: 22, Resistor_SMD:R_0402_1005Metric, symbol Device:R_Small
- added R55, R56: 5.1k, Resistor_SMD:R_0603_1608Metric, symbol Device:R_Small
- added R57: 47, Resistor_SMD:R_0603_1608Metric, symbol Device:R_Small
- added R58, R59: 4.7k, Resistor_SMD:R_0603_1608Metric, symbol Device:R_Small
- added U2: STM32H723ZGTx, Package_QFP:LQFP-144_20x20mm_P0.5mm, symbol MCU_ST_STM32H7:STM32H723ZGTx
- added U3: TPS7A2033PDQNR, Package_SON:Texas_X2SON-4_1x1mm_P0.65mm, symbol Regulator_Linear:TPS7A20xxxDQN
Connections:
- new net: C122.1, C123.2, R57.1, U2.32 (VREF+)
- new net: C115.1, U2.71 (VCAP)
- new net: C116.1, U2.106 (VCAP)
- new net: JP1.1 (A), R47.2, U2.138 (BOOT0)
- new net: R49.1, U2.80 (PD11)
- new net: R50.1, U2.81 (PD12)
- new net: R51.1, U2.82 (PD13)
- new net: J7.B5 (CC2), R56.2
- new net: J7.A5 (CC1), R55.2
- new net: J7.A4 (VBUS), J7.A9 (VBUS), J7.B4 (VBUS), J7.B9 (VBUS)
- new net +3.3VAMCU: C113.1, C121.1, FB3.2, R57.2, U2.33 (VDDA)
- new net +3.3VMCU: C100.1, C101.1, C102.1, C103.1, C104.1, C105.1, C107.1, C108.1, C109.1, C111.1, C112.1, C114.1, C119.1, C120.1, C52.1, C54.1, FB3.1, J6.1 (Pin_1), J8.1 (Pin_1), JP1.2 (B), R58.2, R59.2, U2.108 (VDD), U2.121 (VDD), U2.131 (VDD), U2.144 (VDD), U2.17 (VDD), U2.30 (VDD), U2.39 (VDD), U2.52 (VDD), U2.6 (VBAT), U2.62 (VDD), U2.72 (VDD), U2.84 (VDD), U2.95 (VDD33USB), U3.1 (OUT)
- new net +5.39574468085V: C117.1, C118.1, U3.3 (EN), U3.4 (IN)
- new net +9V: J5.16 (Pin_16)
- new net AIN1: J5.7 (Pin_7), U2.60 (PE9)
- new net AIN2: J5.8 (Pin_8), U2.64 (PE11)
- new net BICK_{ADC}: U2.20 (PF8)
- new net BICK_{DAC}: R49.2
- new net BIN1: J5.9 (Pin_9), U2.66 (PE13)
- new net BIN2: J5.10 (Pin_10), U2.67 (PE14)
- new net CLK_44.1_EN: U2.127 (PG12)
- new net CLK_48_EN: U2.128 (PG13)
- new net CLK_EN: U2.126 (PG11)
- new net EN: J5.15 (Pin_15), U2.68 (PE15)
- new net GNDD: C100.2, C101.2, C102.2, C103.2, C104.2, C105.2, C107.2, C108.2, C109.2, C111.2, C112.2, C113.2, C114.2, C115.2, C116.2, C117.2, C118.2, C119.2, C120.2, C121.2, C122.2, C123.1, C52.2, C54.2, J5.11 (Pin_11), J5.12 (Pin_12), J6.5 (Pin_5), J6.6 (Pin_6), J6.7 (Pin_7), J6.8 (Pin_8), J7.A1 (GND), J7.A12 (GND), J7.B1 (GND), J7.B12 (GND), J7.S1 (SHIELD), J8.4 (Pin_4), JP2.1 (A), R47.1, R55.1, R56.1, U2.107 (VSS), U2.120 (VSS), U2.130 (VSS), U2.143 (PDR_ON), U2.16 (VSS), U2.31 (VSSA), U2.38 (VSS), U2.51 (VSS), U2.61 (VSS), U2.83 (VSS), U2.94 (VSS), U3.2 (GND), U3.5 (Pad)
- new net GPIO0: J5.5 (Pin_5), U2.58 (PE7)
- new net GPIO1: J5.6 (Pin_6), U2.59 (PE8)
- new net INT_{ADC}: U2.129 (PG14)
- new net LRCK_{ADC}: U2.124 (PG9)
- new net LRCK_{DAC}: R50.2
- new net MLCK_{MCU}: U2.99 (PC9)
- new net NRST: J6.4 (Pin_4), JP2.2 (B), U2.25 (NRST)
- new net PDN_{DAC}: U2.87 (PG2)
- new net POT_0: J5.3 (Pin_3), U2.53 (PF13)
- new net POT_1: J5.4 (Pin_4), U2.54 (PF14)
- new net SCL: R58.1, U2.69 (PB10)
- new net SDA: R59.1, U2.70 (PB11)
- new net SDATA_{ADC}: U2.125 (PG10)
- new net SDATA_{DAC}: R51.2
- new net SPDIFRX1: J5.1 (Pin_1), U2.44 (PC4)
- new net SPDIFRX2: J5.2 (Pin_2), U2.45 (PC5)
- new net SWCLK: J6.3 (Pin_3), U2.109 (PA14(JTCK)
- new net SWDIO: J6.2 (Pin_2), U2.105 (PA13(JTMS)
- new net UART_RX: J8.3 (Pin_3), U2.35 (PA1)
- new net UART_TX: J8.2 (Pin_2), U2.34 (PA0)
- new net USB_DN: J7.A7 (D-), J7.B7 (D-), U2.103 (PA11)
- new net USB_DP: J7.A6 (D+), J7.B6 (D+), U2.104 (PA12)
- no-connect marks 0 -> 72
Changed lines of the file:
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@@
 	(generator "eeschema")
 	(generator_version "9.0")
-	(paper "A4")
-)
+	(paper "A3")
