File: object67/object67.kicad_pcb (KiCad board)
At the start: 4 copper layers, 198.2 x 92 mm, 188 parts, among them IC1 AK4493SEQ, IC10 OPA1612AIDRGR, IC2 TAA5242IRGER, IC3 LMK1C1104PWR, IC4 TPA6120A2DWPR, IC5 TPS7A4701RGWT, IC6 TPS7A3301RGWR, IC7 OPA1612AIDRGR, IC8 OPA1612AIDRGR, IC9 OPA1612AIDRGR, J1 SN37A12B, J2 PJ-037A, J3 Power In, J4 216700-0249, J5 216700-0249, J6 Conn_02x08_Odd_Even, U1 RCJ-2223, U10 ADP5070AREZ, U11 TPS62912, U5 RCJ-2223, U7 TPS7A2050PDQNR, U8 TPS7A2033PDQNR, U9 TPS7A2033PDQNR, Y3 ASDLJ-E-49.152MHZ-L-R-T, Y4 ASDLJ-E-45.1584MHz-L-R-T

Commit message: LAyout
Parts:
- removed J4: 216700-0249, object67:2167000249
- removed TPMCLK: TestPoint, TestPoint:TestPoint_Pad_D1.0mm
- added C100: 0.1u, Capacitor_SMD:C_0402_1005Metric, F.Cu at (219.4, 172.6)
- added C101: 0.1u, Capacitor_SMD:C_0402_1005Metric, F.Cu at (211.8, 149.5)
- added C102: 0.1u, Capacitor_SMD:C_0402_1005Metric, F.Cu at (196.4, 166.8)
- added C103: 0.1u, Capacitor_SMD:C_0402_1005Metric, F.Cu at (200.5, 174.0)
- added C104: 0.1u, Capacitor_SMD:C_0402_1005Metric, F.Cu at (221.5, 164.8)
- added C105: 0.1u, Capacitor_SMD:C_0402_1005Metric, F.Cu at (206.0, 149.5)
- added C107: 0.1u, Capacitor_SMD:C_0402_1005Metric, F.Cu at (207.2, 174.0)
- added C108: 0.1u, Capacitor_SMD:C_0402_1005Metric, F.Cu at (219.5, 151.0)
- added C109: 0.1u, Capacitor_SMD:C_0402_1005Metric, F.Cu at (221.5, 159.5)
- added C111: 0.1u, Capacitor_SMD:C_0402_1005Metric, F.Cu at (212.5, 174.5)
- added C112: 0.1u, Capacitor_SMD:C_0402_1005Metric, F.Cu at (200.5, 149.5)
- added C113: 0.1u, Capacitor_SMD:C_0402_1005Metric, F.Cu at (196.5, 169.8)
- added C114: 10u, Capacitor_SMD:CP_Elec_4x5.3, F.Cu at (199.4, 179.8)
- added C115: 2.2u, Capacitor_SMD:C_0603_1608Metric, F.Cu at (218.2, 174.5)
- added C116: 2.2u, Capacitor_SMD:C_0603_1608Metric, F.Cu at (221.5, 153.8)
- added C117: 10u, Capacitor_SMD:C_0603_1608Metric, F.Cu at (186.8, 181.8)
- added C118: 0.1u, Capacitor_SMD:C_0603_1608Metric, F.Cu at (188.5, 181.8)
- added C119: 0.1u, Capacitor_SMD:C_0603_1608Metric, F.Cu at (192.2, 181.0)
- added C120: 10u, Capacitor_SMD:C_0603_1608Metric, F.Cu at (194.0, 181.0)
- added C121: 1u, Capacitor_SMD:C_1206_3216Metric, F.Cu at (192.8, 173.0)
- added C122: 0.1u, Capacitor_SMD:C_0402_1005Metric, F.Cu at (195.4, 168.8)
- added C123: 2.2u, Capacitor_SMD:C_0603_1608Metric, F.Cu at (194.0, 168.4)
- added C52: 0.1u, Capacitor_SMD:C_0402_1005Metric, F.Cu at (196.5, 160.5)
- added C54: 0.1u, Capacitor_SMD:C_0402_1005Metric, F.Cu at (196.5, 155.0)
- added FB3: 120R, Inductor_SMD:L_0603_1608Metric, F.Cu at (195.0, 171.5)
- added J7: USB_C_Receptacle_USB2.0_16P, Connector_USB:USB_C_Receptacle_GCT_USB4085, F.Cu at (152.1, 153.8)
- added J8: Conn_01x04_Pin, Connector_PinHeader_2.54mm:PinHeader_1x04_P2.54mm_Vertical, F.Cu at (148.0, 149.4)
- added JP1: Boot0, Jumper:SolderJumper-2_P1.3mm_Open_RoundedPad1.0x1.5mm, F.Cu at (203.0, 143.8)
- added JP2: NRST, Jumper:SolderJumper-2_P1.3mm_Open_RoundedPad1.0x1.5mm, F.Cu at (190.8, 164.2)
- added R47: 10k, Resistor_SMD:R_0603_1608Metric, F.Cu at (204.0, 146.2)
- added R48: 22, Resistor_SMD:R_0402_1005Metric, F.Cu at (230.5, 140.0)
- added R49: 22, Resistor_SMD:R_0402_1005Metric, F.Cu at (221.5, 167.8)
- added R50: 22, Resistor_SMD:R_0402_1005Metric, F.Cu at (221.5, 166.8)
- added R51: 22, Resistor_SMD:R_0402_1005Metric, F.Cu at (221.5, 165.8)
- added R52: 22, Resistor_SMD:R_0402_1005Metric, F.Cu at (238.0, 127.0)
- added R53: 22, Resistor_SMD:R_0402_1005Metric, F.Cu at (238.0, 128.0)
- added R54: 22, Resistor_SMD:R_0402_1005Metric, F.Cu at (238.0, 129.0)
- added R55: 5.1k, Resistor_SMD:R_0603_1608Metric, F.Cu at (154.8, 155.4)
- added R56: 5.1k, Resistor_SMD:R_0603_1608Metric, F.Cu at (150.4, 163.0)
- added R57: 47, Resistor_SMD:R_0603_1608Metric, F.Cu at (190.8, 170.5)
- added R58: 4.7k, Resistor_SMD:R_0603_1608Metric, F.Cu at (214.9, 179.5)
- added R59: 4.7k, Resistor_SMD:R_0603_1608Metric, F.Cu at (217.5, 177.5)
- added TP10: TestPoint, TestPoint:TestPoint_Pad_D1.0mm, F.Cu at (231.4, 135.5)
- added U2: STM32H723ZGTx, Package_QFP:LQFP-144_20x20mm_P0.5mm, F.Cu at (208.8, 161.8)
- added U3: TPS7A2033PDQNR, Package_SON:Texas_X2SON-4_1x1mm_P0.65mm, F.Cu at (190.3, 181.6)
- C3: footprint Capacitor_THT:CP_Radial_D8.0mm_P3.50mm -> Capacitor_THT:CP_Radial_D8.0mm_P5.00mm
- J5: value 216700-0249 -> Conn_01x16_Socket; footprint object67:2167000249 -> Connector_JST:JST_PH_S16B-PH-K_1x16_P2.00mm_Horizontal
- J6: value Conn_02x08_Odd_Even -> Conn_01x08_Pin; footprint Connector_PinHeader_2.54mm:PinHeader_2x08_P2.54mm_Vertical -> Connector_PinHeader_2.54mm:PinHeader_1x08_P2.54mm_Vertical
- R46: footprint Capacitor_SMD:C_0201_0603Metric -> Resistor_SMD:R_0402_1005Metric
- moved J5 70.0 mm to (190.5, 193.2), turned to 0 degrees
- moved C67 28.9 mm to (225.9, 192.5)
- moved C68 28.9 mm to (227.7, 192.5)
- moved U9 28.7 mm to (229.6, 192.6)
- moved C69 28.7 mm to (231.5, 192.0)
- moved C70 28.7 mm to (233.2, 192.0)
- moved J6 23.9 mm to (166.0, 145.4), turned to -90 degrees
- moved R46 19.7 mm to (225.5, 140.0), turned to 180 degrees
- moved C85 16.2 mm to (177.3, 185.2)
- moved C86 16.2 mm to (179.6, 185.2)
- moved FB4 12.6 mm to (175.4, 187.1), turned to 90 degrees
- moved C59 12.5 mm to (248.6, 192.3)
- moved C60 12.5 mm to (250.6, 192.3)
- moved C62 12.3 mm to (254.3, 192.3)
- moved C61 12.3 mm to (256.0, 192.3)
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- renumbered TPFILOUTLP to TP20, FILOUTRP to TP21, FILOUTLN to TP22, FILOUTRN to TP23, +16 to TP3, -16 to TP4, TPLP to TP5, TPLN to TP6, TPRN to TP7, TPRP to TP8
Connections:
- C72 pad 2: +9V -> VIN
- C78 pad 2: +9V -> VIN
- C79 pad 2: +9V -> VIN
- C80 pad 2: +9V -> VIN
- IC1 pad 46: Net-(IC1-MCLK) -> MLCK_{DAC}
- IC2 pad 2: BICK_{ADC} -> Net-(IC2-BCLK)
- IC2 pad 3: LRCK_{ADC} -> Net-(IC2-FSYNC)
- IC2 pad 4: SDATA_{ADC} -> Net-(IC2-DOUT)
- J2 pad 2: +9V -> VIN
- J3 pad 1: +9V -> VIN
- J5 pad 1: +3.3V -> SPDIFRX1
- J5 pad 10: GND -> BIN2
- J5 pad 13: GND -> unconnected-(J5-Pin_13-Pad13)
- J5 pad 14: GND -> unconnected-(J5-Pin_14-Pad14)
- J5 pad 15: GND -> EN
- J5 pad 16: +3.3V -> VIN
- J5 pad 2: +3.3V -> SPDIFRX2
- J5 pad 3: BICK_{ADC} -> POT_0
- J5 pad 4: LRCK_{ADC} -> POT_1
- J5 pad 5: SDATA_{ADC} -> GPIO0
- J5 pad 6: INT_{ADC} -> GPIO1
- J5 pad 7: GND -> AIN1
- J5 pad 8: GND -> AIN2
- J5 pad 9: GND -> BIN1
- J6 pad 1: +3.3V -> +3.3VMCU
- J6 pad 2: +3.3V -> SWDIO
- J6 pad 3: +3.3V -> SWCLK
- J6 pad 4: BICK_{ADC} -> NRST
- J6 pad 5: PDN_{DAC} -> GND
- J6 pad 6: LRCK_{ADC} -> GND
- J6 pad 7: BICK_{DAC} -> GND
- J6 pad 8: SDATA_{ADC} -> GND
- R46 pad 1: MLCK_{DAC} -> CLK_{45.1584M}
- R46 pad 2: Net-(IC1-MCLK) -> Net-(Y4-OUTPUT)
- U10 pad 11: unconnected-(U10-EN2-Pad11) -> +3.3VMCU
- U10 pad 17: +9V -> VIN
- U10 pad 18: +9V -> VIN
- U10 pad 19: +9V -> VIN
- U10 pad 9: unconnected-(U10-EN1-Pad9) -> +3.3VMCU
- U11 pad 1: +9V -> VIN
- U11 pad 6: +9V -> VIN
- Y3 pad 3: CLK_{45.1584M} -> Net-(Y3-OUTPUT)
- Y4 pad 3: CLK_{45.1584M} -> Net-(Y4-OUTPUT)
Routing:
- net +3.3VMCU: track 0.00 -> 330.2 mm, vias 0 -> 31
- net VIN: track 0.00 -> 109.5 mm, vias 0 -> 13
- net +5.39574468085V: track 0.00 -> 91.6 mm, vias 0 -> 22
- net BICK_{ADC}: track 0.00 -> 68.7 mm, vias 0 -> 2
- net USB_DP: track 0.00 -> 68.1 mm, vias 0 -> 1
- net USB_DN: track 0.00 -> 68.0 mm, vias 0 -> 1
- net SWCLK: track 0.00 -> 62.9 mm, vias 0 -> 1
- net UART_TX: track 0.00 -> 60.1 mm, vias 0 -> 2
- net SWDIO: track 0.00 -> 60.0 mm, vias 0 -> 1
- net UART_RX: track 0.00 -> 59.8 mm, vias 0 -> 2
- net INT_{ADC}: track 0.00 -> 57.8 mm, vias 0 -> 2
- net LRCK_{ADC}: track 0.00 -> 48.9 mm, vias 0 -> 2
- net NRST: track 0.00 -> 47.9 mm
- net SDATA_{ADC}: track 0.00 -> 47.4 mm
- net SDA: track 0.00 -> 34.9 mm, vias 0 -> 2
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- added copper zone on F.Cu, net +15V
- added copper zone on F.Cu, net +16V
- added copper zone on F.Cu, net +3.3V
- added copper zone on F.Cu, net +3.3VA
- added copper zone on F.Cu, net +3.3VMCU
- added copper zone on In2.Cu, net +3.3VMCU
- added copper zone on F.Cu, net +5.39574468085V
- added copper zone on In2.Cu, net +5.39574468085V
- added copper zone on F.Cu, net +5VA
- added copper zone on F.Cu, net -15V
- added copper zone on F.Cu, net -16V
- added copper zone on F.Cu, net Net-(D1-A)
- added copper zone on F.Cu, net Net-(D2-K)
- added copper zone on F.Cu, net Net-(U11-VO)
- added copper zone on F.Cu, net VIN
- added copper zone on In2.Cu, net VIN
