File: object67/object67.kicad_pcb (KiCad board)
At the start: 4 copper layers, 198.2 x 92 mm, 231 parts, among them IC1 AK4493SEQ, IC10 OPA1612AIDRGR, IC2 TAA5242IRGER, IC3 LMK1C1104PWR, IC4 TPA6120A2DWPR, IC5 TPS7A4701RGWT, IC6 TPS7A3301RGWR, IC7 OPA1612AIDRGR, IC8 OPA1612AIDRGR, IC9 OPA1612AIDRGR, J1 SN37A12B, J2 PJ-037A, J3 Power In, J5 Conn_01x16_Socket, J6 Conn_01x08_Pin, J7 USB_C_Receptacle_USB2.0_16P, J8 Conn_01x04_Pin, U1 RCJ-2223, U10 ADP5070AREZ, U11 TPS62912, U2 STM32H723ZGTx, U3 TPS7A2033PDQNR, U5 RCJ-2223, U7 TPS7A2050PDQNR, U8 TPS7A2033PDQNR, U9 TPS7A2033PDQNR, Y3 ASDLJ-E-49.152MHZ-L-R-T, Y4 ASDLJ-E-45.1584MHz-L-R-T

Commit message: Test via stitching
Parts:
- moved R31 16.4 mm to (315.1, 190.4), turned to 90 degrees
- moved C87 11.6 mm to (290.8, 115.8)
- moved C88 11.6 mm to (285.8, 117.2)
- moved C90 11.6 mm to (285.7, 122.2)
- moved IC6 11.6 mm to (276.2, 120.4)
- moved C89 11.6 mm to (273.7, 114.1)
- moved C91 11.6 mm to (275.0, 124.2)
- moved C92 11.6 mm to (276.3, 114.2)
- moved C93 11.6 mm to (271.8, 120.8)
- moved IC5 11.6 mm to (290.2, 120.0)
- moved R44 11.6 mm to (274.6, 125.9)
- moved R45 11.6 mm to (278.4, 125.9)
- moved C50 6.37 mm to (315.4, 166.4)
- moved TP23 4.85 mm to (293.7, 184.1)
- moved R23 4.25 mm to (302.3, 177.3)
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Routing:
- net AOUTRN2: track 0.00 -> 88.4 mm, vias 0 -> 2
- net AOUTRP2: track 0.00 -> 81.5 mm, vias 0 -> 2
- net AOUTLP2: track 0.00 -> 73.4 mm, vias 0 -> 2
- net AOUTLN2: track 0.00 -> 71.4 mm
- net LL: track 0.00 -> 53.4 mm
- net LR: track 0.00 -> 46.9 mm, vias 0 -> 1
- net +15V: track 0.00 -> 43.0 mm, vias 0 -> 10
- net -15V: track 0.00 -> 37.5 mm, vias 0 -> 11
- net HOR: track 0.00 -> 31.9 mm, vias 0 -> 2
- net HOL: track 0.00 -> 30.8 mm, vias 0 -> 2
- net Net-(J1-PadR): track 0.00 -> 21.8 mm
- net GND: track 15.4 -> 27.4 mm, vias 0 -> 6
- net OPA15: track 0.00 -> 9.82 mm, vias 0 -> 2
- net OPA21: track 0.00 -> 8.62 mm, vias 0 -> 2
- net OPA20: track 0.00 -> 7.16 mm
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- added copper zone on In1.Cu, net GND

Commit message: Skibidi
Routing:
- net +3.3V: track 24.0 -> 141.2 mm, vias 5 -> 9
- net GND: track 27.4 -> 41.0 mm, vias 6 -> 17
- added copper zone on In2.Cu, net +3.3V
- removed copper zone on In1.Cu, net GND

Commit message: done
Parts:
- moved TP20 15.3 mm to (286.2, 158.0)
- moved TP22 15.1 mm to (286.6, 148.9)
- moved TP21 7.73 mm to (294.7, 178.6)
- moved R1 7.11 mm to (245.8, 180.5), turned to 0 degrees
- moved TP3 4.24 mm to (175.8, 111.9)
- moved TP8 3.64 mm to (259.4, 176.7)
- moved TP7 2.22 mm to (259.4, 171.6)
- moved TP23 1.70 mm to (294.8, 182.8)
- moved TP4 1.57 mm to (176.9, 132.2), turned to 180 degrees
- moved TP6 0.67 mm to (261.2, 152.2)
- moved TP5 0.51 mm to (261.1, 146.0)
Routing:
- net +15V: track 43.0 -> 148.5 mm, vias 10 -> 21
- net -15V: track 37.5 -> 136.1 mm, vias 11 -> 22
- net AINLP: track 0.00 -> 88.5 mm
- net +5VA: track 29.6 -> 114.5 mm, vias 5 -> 4
- net +3.3VA: track 19.1 -> 102.9 mm, vias 5 -> 4
- net AINRP: track 0.00 -> 83.5 mm
- net +3.3V: track 141.2 -> 173.4 mm, vias 9 -> 10
- net +16V: track 6.21 -> 29.0 mm, vias 2 -> 18
- net +5.39574468085V: track 91.6 -> 114.3 mm
- net -16V: track 2.96 -> 23.1 mm, vias 2 -> 17
- net VIN: track 109.5 -> 128.9 mm
- net GND: track 41.0 -> 54.2 mm, vias 17 -> 25
- net +5VREFR: track 14.9 -> 19.2 mm
- net AOUTRP: track 28.0 -> 30.9 mm
- net AOUTLP: track 29.6 -> 32.4 mm
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- added copper zone on In2.Cu, net +15V
- added copper zone on In2.Cu, net +16V
- added copper zone on In2.Cu, net -15V
- added copper zone on In2.Cu, net -16V
- added copper zone on B.Cu, net GND
- added copper zone on F.Cu, net GND
- added copper zone on In1.Cu, net GND

Commit message: done
Routing:
- net GND: vias 25 -> 33
Changed lines of the file:
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@@
+	)
+	(via
+		(at 224.5 164.4)
+		(size 0.6)
+		(drill 0.3)
+		(layers "F.Cu" "B.Cu")
+		(free yes)
+		(net 147)
+	)
+	(via
+		(at 224.5 165.6)
+		(size 0.6)
+		(drill 0.3)
+		(layers "F.Cu" "B.Cu")
+		(free yes)
+		(net 147)
+	)
+	(via
+		(at 226.3 164.4)
+		(size 0.6)
+		(drill 0.3)
+		(layers "F.Cu" "B.Cu")
+		(free yes)
+		(net 147)
 	)
 	(via
@@
 		(drill 0.3)
 		(layers "F.Cu" "B.Cu")
+		(net 147)
+	)
+	(via
+		(at 220.9 156.8)
+		(size 0.6)
+		(drill 0.3)
+		(layers "F.Cu" "B.Cu")
+		(free yes)
 		(net 147)
 	)
@@
 	)
 	(via
+		(at 161.9 185.6)
+		(size 0.6)
+		(drill 0.3)
+		(layers "F.Cu" "B.Cu")
+		(free yes)
+		(net 147)
+	)
+	(via
 		(at 201.7 149.5)
 		(size 0.45)
@@
 	)
 	(via
+		(at 220.9 155.7)
+		(size 0.6)
+		(drill 0.3)
+		(layers "F.Cu" "B.Cu")
+		(free yes)
+		(net 147)
+	)
+	(via
 		(at 199.5 168.1)
 		(size 0.45)
@@
 	)
 	(via
+		(at 226.3 165.6)
+		(size 0.6)
+		(drill 0.3)
+		(layers "F.Cu" "B.Cu")
+		(free yes)
+		(net 147)
+	)
+	(via
 		(at 241.4 161.5)
 		(size 0.6)
@@
 		(drill 0.3)
 		(layers "F.Cu" "B.Cu")
+		(net 147)
+	)
+	(via
+		(at 221.8 156.2)
+		(size 0.6)
+		(drill 0.3)
+		(layers "F.Cu" "B.Cu")
+		(free yes)
 		(net 147)
 	)
@@
 	)
 	(zone
-		(net 147)
-		(net_name "GND")
-		(layer "F.Cu")
-		(hatch edge 0.5)
-		(connect_pads yes
-			(clearance 0.25)
-		)
-		(min_thickness 0.25)
-		(filled_areas_thickness no)
-		(fill yes
-			(thermal_gap 0.25)
-			(thermal_bridge_width 0.25)
-		)
-		(polygon
-			(pts
-				(xy 144.8 105.6) (xy 348.4 104.9) (xy 345.8 202.2) (xy 141.8 206.9)
-			)
-		)
-	)
-	(zone
 		(net 32)
 		(net_name "+5.39574468085V")
@@
 			(pts
 				(xy 165.4 125.6) (xy 168.4 125.6) (xy 168.4 129.6) (xy 165.4 129.6)
+			)
+		)
+	)
+	(zone
+		(net 147)
+		(net_name "GND")
+		(layers "F.Cu" "B.Cu" "In1.Cu")
+		(hatch edge 0.5)
+		(connect_pads yes
+			(clearance 0.25)
+		)
+		(min_thickness 0.25)
+		(filled_areas_thickness no)
+		(fill yes
+			(thermal_gap 0.5)
+			(thermal_bridge_width 0.5)
+		)
+		(polygon
+			(pts
+				(xy 143.1 106.2) (xy 135.2 204.4) (xy 357 205.7) (xy 351 101.1)
 			)
 		)
@@
 			)
 		)
-	)
-	(zone
-		(net 147)
-		(net_name "GND")
-		(layer "B.Cu")
-		(name "5V Power Supply")
-		(hatch edge 0.5)
-		(priority 35)
-		(connect_pads yes
-			(clearance 0.25)
-		)
-		(min_thickness 0.25)
-		(filled_areas_thickness no)
-		(fill yes
-			(thermal_gap 0.25)
-			(thermal_bridge_width 0.3)
-			(island_removal_mode 1)
-			(island_area_min 10)
-		)
-		(polygon
-			(pts
-				(xy 142.4 105.4) (xy 358.1 105.8) (xy 354.4 211.3) (xy 140.5 210.4)
-			)
-		)
-	)
-	(zone
-		(net 147)
-		(net_name "GND")
-		(layer "In1.Cu")
-		(hatch edge 0.5)
-		(priority 1)
-		(connect_pads yes
-			(clearance 0.25)
-		)
-		(min_thickness 0.25)
-		(filled_areas_thickness no)
-		(fill yes
-			(thermal_gap 0.25)
-			(thermal_bridge_width 0.3)
-			(island_removal_mode 1)
-			(island_area_min 10)
-		)
-		(polygon
-			(pts
-				(xy 143 105.2) (xy 360.4 103.7) (xy 357.5 211.5) (xy 137.4 208.8)
-			)
-		)

Commit message: done
Routing:
- net GND: vias 33 -> 414
Other:
- outline, holes or cut-outs redrawn
- board text added: "AK4493SEQ HiFi DSP Audio Test Board Rev.1"
- board text added: "{ "ViaStitching": "0.2", "stitch_zone_0": { "HSpacing": "5", "VSpacing": "5", "HOffset": "0", "VOffset": "0", "Clearance": "0.25", "Randomize": false } }"
