File: object67/xsp_main.kicad_sch (KiCad schematic)
At the start: 67 parts, among them IC5 TPS7A4701RGWT, IC6 TPS7A3301RGWR, J2 PJ-037A, J3 Power In, J4 216700-0249, J5 216700-0249, J6 Conn_02x08_Odd_Even, U10 ADP5070AREZ, U11 TPS62912, U7 TPS7A2050PDQNR, U8 TPS7A2033PDQNR, U9 TPS7A2033PDQNR

Commit message: LAyout
Parts:
- removed J4, J5: 216700-0249, object67:2167000249, symbol object67:216700-0249
- removed J6: Conn_02x08_Odd_Even, Connector_PinHeader_2.54mm:PinHeader_2x08_P2.54mm_Vertical, symbol Connector_Generic:Conn_02x08_Odd_Even
Connections:
- net +3.3VMCU: now reaches U10.11 (EN2)
- net +3.3VMCU: now also U10.9 (EN1)
- no-connect marks 34 -> 22
